File: KiCad/Easy_Z80.sch (KiCad schematic (older format))
At the start: 58 parts, among them J1 POWER, J2 SERIAL_A, J3 SERIAL_B, J4 VBAT, J5 RC2014_BUS, J6 RC2014_EXT, J7 RC2014_SPARE, SW1 RESET, U1 Z84C00, U10 74HCT670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

Commit message: KiCad: Replace files with version 1.1
Signed-off-by: Sergey Kiselev <skiselev@gmail.com>
Parts:
- removed C15: 100n, My_Components:Cap_Cer_508, symbol C
- removed RR1, RR2, RR3: 4.7k, My_Components:Conn_SIL5, symbol RR4
- added RN1, RN2, RN3: 4.7k, My_Components:Conn_SIL5, symbol Device:R_Network04
- added RN4: 4.7k, My_Components:Conn_SIL9, symbol Device:R_Network08
- C1, C10, C11, C12, C13, C14, C16, C17, C18, C19, C2, C20, C21, C22, C23, C3, C4, C5, C6, C7, C8, C9: symbol C -> Device:C
- C24: symbol CP1 -> Device:CP1
- D1: symbol LED -> Device:LED
- J1: symbol Jack-DC -> Connector:Barrel_Jack_Switch
- J2, J3: symbol DE9 -> my_components:DE9
- J4: symbol Conn_01x02 -> Connector_Generic:Conn_01x02
- J5: symbol Conn_01x39 -> Connector_Generic:Conn_01x39
- J6: symbol Conn_01x10 -> Connector_Generic:Conn_01x10
- J7: symbol Conn_01x05 -> Connector_Generic:Conn_01x05
- JP1, JP2: symbol Jumper_NC_Dual -> Device:Jumper_NC_Dual
- QG1, QG2: symbol OSC_Half_Can -> my_components:OSC_Half_Can
- R1, R2, R3, R4, R5: symbol R -> Device:R
- RV1: symbol POT -> Device:R_POT
- SW1: symbol Switch_Tactile_Vertical -> my_components:Switch_Tactile_Vertical
- U1: symbol Z84C00 -> my_components:Z84C00
- U10, U11: value 74HCT670 -> 74HC670; symbol 74HCT670 -> my_components:74HCT670
- U12: value 74HCT74 -> 74HC74; symbol 74LS74 -> my_components:74LS74
- U2: symbol Z84C30 -> my_components:Z84C30
- U3: symbol Z84C40 -> my_components:Z84C40
- U4: symbol AS6C4008_PWR-RESCUE-Easy_Z80 -> my_components:AS6C4008_PWR
- U5: symbol SST39SF040 -> my_components:SST39SF040
- U6: symbol ADM693 -> my_components:ADM693
- U7, U8: symbol MAX232 -> my_components:MAX232
- U9: symbol ATF16V8B -> my_components:ATF16V8B
Connections:
- net D0: now also RN4.2 (R1)
- net D1: now also RN4.3 (R2)
- net D2: now also RN4.4 (R3)
- net D3: now also RN4.5 (R4)
- net D4: now also RN4.6 (R5)
- net D5: now also RN4.7 (R6)
- net D6: now also RN4.8 (R7)
- net D7: now also RN4.9 (R8)
- net GND: now also J2.GND, J3.GND, RN2.1 (common), RN3.1 (common)
- net MA14: now also RN2.4 (R3)
- net MA15: now also RN2.5 (R4)
- net MA16: now also RN2.3 (R2)
- net MA17: now also RN2.2 (R1)
- net MA18: now also RN3.4 (R3)
- net MA19: now also RN3.5 (R4)
- net MA20: now also RN3.3 (R2)
- net MA21: now also RN3.2 (R1)
- net VCC: now also RN1.1 (common), RN4.1 (common)
- net ~BUSREQ: now also RN1.4 (R3)
- net ~INT: now also RN1.2 (R1)
- net ~NMI: now also RN1.3 (R2)
- net ~WAIT: now also RN1.5 (R4)
Other:
- moved on the sheet: J6
